Commit message: camera corrections controller_changes adding hardeware parameters

File: src/example/description/ros2_control_description/robot2.ros2_control.xacro (robot description, xacro)
@@ -13,21 +13,47 @@
         </xacro:unless>
       </hardware>
-      <joint name="left_front_wheel_joint">
-        <state_interface name="position"/>
-        <command_interface name="position"/>
-      </joint>
-      <joint name="right_front_wheel_joint">
-        <state_interface name="position"/>
-        <command_interface name="position"/>
-      </joint>
-      <joint name="left_rear_wheel_joint">
-        <state_interface name="velocity"/>
-        <state_interface name="position"/>
+      <joint name="front_wheels_joint">
+        <state_interface name="temperature_front_left"/>
+        <state_interface name="temperature_front_right"/>
+        <state_interface name="temperature_front_timestampt"/>
+        <state_interface name="velocity_front_left"/>
+        <state_interface name="velocity_front_right"/>
+        <state_interface name="velocity_front_timestamp"/>
+        <state_interface name="throttle_front_left"/>
+        <state_interface name="throttle_front_right"/>
+        <state_interface name="throttle_front_timestamp"/>
+        <state_interface name="reverse_front_left"/>
+        <state_interface name="reverse_front_right"/>
+        <state_interface name="reverse_front_timestamp"/>
+        <state_interface name="brake_front_left"/>
+        <state_interface name="brake_front_right"/>
+        <state_interface name="brake_front_timestamp"/>
         <command_interface name="velocity"/>
       </joint>
-      <joint name="right_rear_wheel_joint">
-        <state_interface name="velocity"/>
-        <state_interface name="position"/>
+      <joint name="rear_wheels_joint">
+        <state_interface name="temperature_rear_left"/>
+        <state_interface name="temperature_rear_right"/>
+        <state_interface name="temperature_rear_timestamp"/>
+        <state_interface name="velocity_rear_left"/>
+        <state_interface name="velocity_rear_right"/>
+        <state_interface name="velocity_rear_timestamp"/>
+        <state_interface name="throttle_rear_left"/>
+        <state_interface name="throttle_rear_right"/>
+        <state_interface name="throttle_rear_timestamp"/>
+        <state_interface name="reverse_rear_left"/>
+        <state_interface name="reverse_rear_right"/>
+        <state_interface name="reverse_rear_timestamp"/>
+        <state_interface name="brake_rear_left"/>
+        <state_interface name="brake_rear_right"/>
+        <state_interface name="brake_rear_timestamp"/>
         <command_interface name="velocity"/>
+      </joint>
+      <joint name="direction_joint">
+        <state_interface name="steering_angle"/>
+        <state_interface name="steering_angle_timestamp"/>
+        <state_interface name="steering_torque_high"/>
+        <state_interface name="steering_torque_low"/>
+        <state_interface name="steering_torque_timestamp"/>
+        <command_interface name="direction"/>
       </joint>
     </ros2_control>
@@ -37,21 +63,24 @@
         <hardware>
           <plugin>example/GpsHardware</plugin>
-          <!--
-          <param name="interface_type">serial</param>
-          <param name="serial_device">/dev/ttyUSB0</param>
-          or
-          <param name="interface_type">ethernet</param>
-          <param name="port">4001</param>
-          -->
+          <param name="ip">192.168.1.150</param>
+          <param name="port">16718</param>
         </hardware>
         <sensor name="gps_sensor">
+          <state_interface name="gnss_fix"/>
           <state_interface name="latitude"/>
           <state_interface name="longitude"/>
-          <state_interface name="altitude"/>
-          <!--
-          <state_interface name="velocity_x"/>
-          <state_interface name="velocity_y"/>
+          <state_interface name="height"/>
+          <state_interface name="velocity_north"/>
+          <state_interface name="velocity_east"/>
+          <state_interface name="velocity_down"/>
+          <state_interface name="roll"/>
+          <state_interface name="pitch"/>
           <state_interface name="heading"/>
-          -->
+          <state_interface name="angular_velocity_x"/>
+          <state_interface name="angular_velocity_y"/>
+          <state_interface name="angular_velocity_z"/>
+          <state_interface name="accelerometer_x"/>
+          <state_interface name="accelerometer_y"/>
+          <state_interface name="accelerometer_z"/>
         </sensor>
       </ros2_control>

File: src/example/description/ros2_control_description/robot2_description.xacro (robot description, xacro)
@@ -31,7 +31,6 @@
             <origin xyz="0.0 0.0 0.2" rpy="0.0 0.0 0.0"/>
         </joint>
-        <!-- Rear Wheels -->
-        <!-- left real wheel -->
-        <link name="left_rear_wheel">
+        <!-- Rear Axel -->
+        <link name="rear_wheels">
             <visual>
                 <origin xyz="0.0 0.0 0.0" rpy="1.5708 0.0 1.5708"/>
@@ -56,13 +55,14 @@
             </inertial>
         </link>
-        <joint name="left_rear_wheel_joint" type="continuous">
+        <joint name="rear_wheels_joint" type="continuous">
             <parent link="chassis_link"/>
-            <child link="left_rear_wheel"/>
-            <origin xyz="-0.5 0.3 -0.1" rpy="0.0 0.0 1.5708"/>
+            <child link="rear_wheels"/>
+            <origin xyz="-0.5 0.0 -0.1" rpy="0.0 0.0 1.5708"/>
             <axis xyz="1 0 0"/>
             <limit effort="10.0" velocity="5.0"/>
         </joint>
-        <!-- right rear wheel -->
-        <link name="right_rear_wheel">
+        <!-- Front Axel -->
+        <!-- front wheels -->
+        <link name="front_wheels">
             <visual>
                 <origin xyz="0.0 0.0 0.0" rpy="1.5708 0.0 1.5708"/>
@@ -87,14 +87,12 @@
             </inertial>
         </link>
-        <joint name="right_rear_wheel_joint" type="continuous">
+        <joint name="front_wheels_joint" type="revolute">
             <parent link="chassis_link"/>
-            <child link="right_rear_wheel"/>
-            <origin xyz="-0.5 -0.3 -0.1" rpy="0.0 0.0 1.5708"/>
-            <axis xyz="1 0 0"/>
-            <limit effort="10.0" velocity="5.0"/>
+            <child link="front_wheels"/>
+            <origin xyz="0.5 0.0 -0.1" rpy="0.0 0.0 1.5708"/>
+            <axis xyz="0 0 1"/>
+            <limit lower="-1.57" upper="1.57" effort="10.0" velocity="5.0"/>
         </joint>
-        <!-- Front Wheels -->
-        <!-- left front wheel -->
-        <link name="left_front_wheel">
+        <link name="direction_link">
             <visual>
                 <origin xyz="0.0 0.0 0.0" rpy="1.5708 0.0 1.5708"/>
@@ -119,39 +117,8 @@
             </inertial>
         </link>
-        <joint name="left_front_wheel_joint" type="revolute">
+        <joint name="direction_joint" type="revolute">
             <parent link="chassis_link"/>
-            <child link="left_front_wheel"/>
-            <origin xyz="0.5 0.3 -0.1" rpy="0.0 0.0 1.5708"/>
-            <axis xyz="0 0 1"/>
-            <limit lower="-1.57" upper="1.57" effort="10.0" velocity="5.0"/>
-        </joint>
-        <!-- right front wheel -->
-        <link name="right_front_wheel">
-            <visual>
-                <origin xyz="0.0 0.0 0.0" rpy="1.5708 0.0 1.5708"/>
-                <geometry>
-                    <cylinder radius="0.1" length="0.05"/>
-                </geometry>
-                <material name="black">
-                    <color rgba="0.1 0.1 0.1 1.0"/>
-                </material>
-            </visual>
-            <collision>
-                <origin xyz="0.0 0.0 0.0" rpy="1.5708 0.0 1.5708"/>
-                <geometry>
-                    <cylinder radius="0.1" length="0.05"/>
-                </geometry>
-            </collision>
-            <inertial>
-                <origin xyz="0.0 0.0 0.0" rpy="1.5708 0.0 1.5708"/>
-                <mass value="1.0"/>
-                <inertia ixx="0.01" ixy="0.0" ixz="0.0"
-                         iyy="0.01" iyz="0.0" izz="0.01"/>
-            </inertial>
-        </link>
-        <joint name="right_front_wheel_joint" type="revolute">
-            <parent link="chassis_link"/>
-            <child link="right_front_wheel"/>
-            <origin xyz="0.5 -0.3 -0.1" rpy="0.0 0.0 1.5708"/>
+            <child link="direction_link"/>
+            <origin xyz="0.0 0.0 0.0" rpy="0.0 0.0 0.0"/>
             <axis xyz="0 0 1"/>
             <limit lower="-1.57" upper="1.57" effort="10.0" velocity="5.0"/>

Commit message: Adding the header to the msg for the objects detected. save and read of a anpp file from the gpss system

File: src/example/description/ros2_control_description/robot2.ros2_control.xacro (robot description, xacro)
@@ -1,5 +1,5 @@
 <?xml version="1.0"?>
 <robot xmlns:xacro="http://www.ros.org/wiki/xacro">
-  <xacro:macro name="Robot4Farmers" params="use_sim:=false">
+  <xacro:macro name="Robot4Farmers" params="use_sim:=false file_name:= read:=0">
     <ros2_control name="robot2_hardware" type="system">
       <hardware>
@@ -64,4 +64,6 @@
           <param name="ip">192.168.1.150</param>
           <param name="port">16718</param>
+          <param name="file_name_to_reproduce">$(arg file_name)</param>
+          <param name="read_">$(arg read)</param>
         </hardware>
         <sensor name="gps_sensor">

File: src/example/description/urdf/my_robot.urdf.xacro (robot description, xacro)
@@ -6,4 +6,4 @@
   <xacro:include filename="$(find example)/ros2_control_description/robot2.ros2_control.xacro"/>
   <xacro:Robot4Farmers_description/>
-  <xacro:Robot4Farmers use_sim="false"/>
+  <xacro:Robot4Farmers use_sim="false" file_name:="" read_:0/>
 </robot>

Commit message: way to publish the speed to the controller cleaning of the code and adding of a elements to pass the file name of the gps data to read, in the terminal

File: src/example/description/ros2_control_description/robot2.ros2_control.xacro (robot description, xacro)
@@ -1,5 +1,5 @@
 <?xml version="1.0"?>
 <robot xmlns:xacro="http://www.ros.org/wiki/xacro">
-  <xacro:macro name="Robot4Farmers" params="use_sim:=false file_name:= read:=0">
+  <xacro:macro name="Robot4Farmers" params="use_sim:=false">
     <ros2_control name="robot2_hardware" type="system">
       <hardware>
@@ -64,6 +64,6 @@
           <param name="ip">192.168.1.150</param>
           <param name="port">16718</param>
-          <param name="file_name_to_reproduce">$(arg file_name)</param>
-          <param name="read_">$(arg read)</param>
+          <param name="read">$(optenv GPS_READ 0)</param>
+          <param name="file_name">$(optenv GPS_FILE "")</param>
         </hardware>
         <sensor name="gps_sensor">

File: src/example/description/urdf/my_robot.urdf.xacro (robot description, xacro)
@@ -6,4 +6,4 @@
   <xacro:include filename="$(find example)/ros2_control_description/robot2.ros2_control.xacro"/>
   <xacro:Robot4Farmers_description/>
-  <xacro:Robot4Farmers use_sim="false" file_name:="" read_:0/>
+  <xacro:Robot4Farmers use_sim="false"/>
 </robot>
